Commit message: Final of the robotic arm mycobot_280

File: mycobot_description/urdf/mech/adaptive_gripper.urdf.xacro (robot description, xacro)
@@ -1,12 +1,22 @@
-<?xml version="1.0"?>
-<robot xmlns:xacro="http://www.ros.org/wiki/xacro">
-  <xacro:property name="joint_effort" value="56.0"/>
-  <xacro:property name="joint_velocity" value="2.792527"/>
+<?xml version="1.0"?> <!-- XML declaration -->
+<robot xmlns:xacro="http://www.ros.org/wiki/xacro"> <!-- Robot tag and this two line in any stander URDF files
+   and the Xacro here tells us we are using the xacro macro for more maintainable robot descriptions-->
+  <!--What xacro do is reduce the amoount of code you need to write in each URDF file. It's like a macro
+  consolidating all the code into really tiny modular reusable chunks.-->
+  <!--NOTE:::-->
+  <!-- THIS OVER ALL STRUCTURE, ALL THE URDF FILES DOES IS IT CREATES A GRIPPER_BASE AND A GRIPPER_CONTROLLER WITH SIX SYNCHRONIZED MOVING PARTS IT'S GOT 3 ON EACH SIDE -->
+  <!-- And out gripper movment is controlled by our single main joint the gripper controller-->
+  <!--  -->
+  <!--These are the physical limitation that we're putting on our grippers movement. -->
+  <xacro:property name="joint_effort" value="56.0"/> <!-- How much force our joints can exert which is the maxmum torque the joint can apply-->
+  <xacro:property name="joint_velocity" value="2.792527"/> <!-- How fast the joints will move and we use radians per second-->
   <xacro:property name="joint_damping" value="0.0"/>
   <xacro:property name="joint_friction" value="0.0"/>
-  <xacro:property name="gripper_link_mass" value="0.007"/>
+  <!-- Here we define some mass and inertial properties and these values are very important for accurate physics simulation -->
+  <xacro:property name="gripper_link_mass" value="0.007"/> <!-- How much mass using kilograms -->
   <xacro:property name="gripper_link_ixx" value="1e-6"/>
   <xacro:property name="gripper_link_iyy" value="1e-6"/>
   <xacro:property name="gripper_link_izz" value="1e-6"/>
+  <!-- This is a reusable template for the inertial properties that we use multiple times throughout the robot -->
   <xacro:macro name="gripper_link_inertial">
     <inertial>
@@ -19,27 +29,45 @@
     </inertial>
   </xacro:macro>
+  <!-- Here we have the main gripper definition and this macro take 3 parameters parent,prefix and origin-->
+  <!-- Parent is what the gripper attaches to on your robot-->
+  <!-- Prefix is a namespace prefix for unique naming. And this come in handy if you've got many different grippers or robots on your amr like gripper for a left arm and one for the right arm prefix left and prefix right -->
+  <!-- origin is where the girpper actually mounts-->
   <xacro:macro name="adaptive_gripper" params="parent prefix *origin">
+    <!-- Here we start with the links and as we know any robot is a collection of links and joints and links are the hard rigig pieces and joints are the movable pieces -->
+    <!-- And the first link we define here is the gripper base-->
+    <!-- And as we can see an link has three highlevel parts inertial, Visual and Collision-->
     <link name="${prefix}gripper_base">
+      <!-- First bluck is inertial and it defines the physical properties of the gripper base-->
       <inertial>
-        <origin xyz="0 0 0.0" rpy="0 0 0"/>
-        <mass value="0.07"/>
+        <origin xyz="0 0 0.0" rpy="0 0 0"/> <!-- Like origin and where it's conect-->
+        <mass value="0.07"/> <!-- And its mass (kilograms)-->
         <inertia
           ixx="0.000010725" ixy="0.0" ixz="0.0"
           iyy="0.000014392" iyz="0.0"
           izz="0.000018517"/>
-      </inertial>
+      </inertial> <!-- And it's inertia-->
+      <!-- The second bluck is visual and it defines how the actual grippper looks   -->
       <visual>
         <geometry>
           <mesh filename="file://$(find mycobot_description)/meshes/adaptive_gripper/visual/gripper_base.dae"/>
+          <!--  This mesh file the dae file create the realistic appearance for the robot-->
         </geometry>
         <origin xyz="0.0 0.0 -0.012" rpy="0 0 0"/>
       </visual>
-      <collision>
-        <geometry>
+      <!--The 3rd bluck is the collision and we're using just a simplified shape for the collision, a box. we're modeling the gripper base as an actual box-->
+      <!-- Why we do that? because it's much simpler for physics engines to be able to handle a box geometry than a complicated mesh geometry. it's much more lightweight on different physics engines like Gazebo-->
+      <collision>
+        <geometry>
+          <!-- With the length, width and the height of the box-->
           <box size="0.065 0.025 0.025"/>
+          <!-- But collision uses simple geometic shapes for very efficient collision checking. -->
         </geometry>
         <origin xyz="0.0 0.0 0.0" rpy="0 0 0"/>
       </collision>
-    </link>
+      <!--So in the visual aspect we use the mesh file because the look but for the basic collision we use box or sphere to make it easier and quicker for the simulation engines to decide if two robots are colliding or not-->
+    </link>
+    <!-- Here after our first link we see our first joint-->
+    <!-- And this the joint that conect the parent which is the endeffector of the arm the last piece they often call it the Flange where the gripper actually conects to the robotic arm. -->
+    <!-- And this parent conected to the gribber_base and it's fixed because we normally screw on the gripper base onto the robotic arm. -->
     <joint name="${prefix}${parent}_to_${prefix}gripper_base" type="fixed">
       <parent link="${prefix}${parent}"/>
@@ -137,4 +165,6 @@
       </collision>
     </link>
+    <!-- This joint is the main controll point of the gripper basically it's the motor that mkae the gripper open and close or do it job-->
+    <!-- So the gripper controller will have a joint(a motor) that'll move it and then they will be other links there like the fingers gripper_left2 and so on that will mimic the behavior the movement that occurs at the gripper controller-->
     <joint name="${prefix}gripper_controller" type="revolute">
       <axis xyz="0 0 1"/>
@@ -145,12 +175,16 @@
       <dynamics damping="${joint_damping}" friction="${joint_friction}"/>
     </joint>
+    <!-- And all the other gripper joint are designed to mimic the gripper controller-->
     <joint name="${prefix}gripper_base_to_${prefix}gripper_left2" type="revolute">
-      <axis xyz="0 0 1"/>
-      <limit effort="${joint_effort}" lower="-0.8" upper="0.5" velocity="${joint_velocity}"/>
-      <parent link="${prefix}gripper_base"/>
-      <child link="${prefix}gripper_left2"/>
-      <origin xyz="-0.005 0.027 0" rpy="0 0 0"/>
+      <axis xyz="0 0 1"/> <!-- This define which direction the joint will rotates-->
+      <limit effort="${joint_effort}" lower="-0.8" upper="0.5" velocity="${joint_velocity}"/> <!-- This defines how far the joint can move in radians. And you got joint_velocity which define how fast it can move in radians per second. And all this was defined up in our parameters section-->
+      <parent link="${prefix}gripper_base"/> <!-- This show what parent part is conected to-->
+      <child link="${prefix}gripper_left2"/> <!-- This the child of the joint which is the part that conected to the parent-->
+      <origin xyz="-0.005 0.027 0" rpy="0 0 0"/> <!-- This defines where the joint is located relative to its parent the gripper_base-->
+      <!-- We define the name of the joint that we want to mimic for this paricaular joint and in this case we mimic the gripper controller and we have a multiplier which scales the movement and here it's going to be 1.0
+       so if you move 5 radians on the gripper controller you will move 5 radians on the gripper base to gripper_left2 joint. -->
       <mimic joint="${prefix}gripper_controller" multiplier="1.0" offset="0"/>
       <dynamics damping="${joint_damping}" friction="${joint_friction}"/>
+      <!-- And this is the same structured for all the other joints-->
     </joint>
     <joint name="${prefix}gripper_left3_to_${prefix}gripper_left1" type="revolute">
@@ -160,5 +194,5 @@
       <child link="${prefix}gripper_left1"/>
       <origin xyz="-0.027 0.016 0" rpy="0 0 0"/>
-      <mimic joint="${prefix}gripper_controller" multiplier="-1.0" offset="0"/>
+      <mimic joint="${prefix}gripper_controller" multiplier="-1.0" offset="0"/> <!-- for this one if you move 5 radians on the gripper controller you will move -5 radians on the gripper base to gripper_left1 joint.  -->
       <dynamics damping="${joint_damping}" friction="${joint_friction}"/>
     </joint>
@@ -190,7 +224,8 @@
       <dynamics damping="${joint_damping}" friction="${joint_friction}"/>
     </joint>
+    <!-- This defines gazebo specific element. And gazebo our simulation engine  -->
     <gazebo reference="${prefix}gripper_base">
-      <visual>
-        <material>
+      <visual> <!-- We define here how the gripper should look and appear in Gazebo simulation-->
+        <material> <!-- And this corresponds to a color for the gripper-->
           <ambient>1 1 1 1</ambient>
           <diffuse>1 1 1 1</diffuse>

File: mycobot_description/urdf/mech/g_shape_base_v2_0.urdf.xacro (robot description, xacro)
@@ -1,30 +1,34 @@
 <?xml version="1.0" ?>
 <robot xmlns:xacro="http://wiki.ros.org/xacro">
+    <!-- THIS FILE IS JUST DESCRBING A STATIC BASE PLACE -->
+    <!-- This file define a single macro called g_shape_base and this takes 2 parameters the base_link and a prefix for unique naming-->
     <xacro:macro name="g_shape_base" params="base_link prefix">
+       <!-- In this macro we define a single link with standard URDF components. The inertial, visual and collision-->
         <link name="${prefix}${base_link}">
             <inertial>
-                <origin xyz="0 0 0.0" rpy="0 0 0"/>
-                <mass value="0.33"/>
+                <origin xyz="0 0 0.0" rpy="0 0 0"/> <!-- the origin the position XYZ and the orientation roll pitch and yaw-->
+                <mass value="0.33"/> <!-- The mass of the link in kilograms-->
                 <inertia
                     ixx="0.000784" ixy="0.0" ixz="0.0"
                     iyy="0.000867" iyz="0.0"
                     izz="0.001598"/>
-            </inertial>
-            <visual>
+            </inertial> <!-- The inertia describe how the mass is distributed. it impact how the link resists rotational motion-->
+            <visual> <!-- A visula componnet define the gripper base how should it look like.-->
                 <geometry>
                     <mesh filename="file://$(find mycobot_description)/meshes/g_shape_base_v2_0/visual/base_link.dae"/>
                 </geometry>
-                <origin xyz="0.0 0 -0.03" rpy="0 0 ${pi/2}"/>
+                <origin xyz="0.0 0 -0.03" rpy="0 0 ${pi/2}"/> <!-- This is the origin of the visual component of this link which defines the position and the orientation of the visual representation with offset a little bit -0.03 to make it nice and pretty in visualiztion-->
             </visual>
-            <collision>
-                <geometry>
+            <collision> <!-- Define the geometry that is used to detected if the particular link collides with an object or another part of the robotic arm in gazebo environment-->
+                <geometry> <!-- we define it as a baic box shape length,width and height and it's in meters -->
                     <box size="0.105 0.14 0.02"/>
                 </geometry>
-                <origin xyz="0.0 0.0 -0.015" rpy="0 0 0"/>
+                <origin xyz="0.0 0.0 -0.015" rpy="0 0 0"/> <!-- Here the origin which it aids in how we position that collision geometry within the link. -->
             </collision>
         </link>
+        <!-- This gazebo section to define how the base appears in simulation.-->
         <gazebo reference="${prefix}${base_link}">
             <visual>
-                <material>
+                <material> <!-- And this number define the color and it's gray -->
                     <ambient>0.5 0.5 0.5 1</ambient>
                     <diffuse>0.5 0.5 0.5 1</diffuse>

File: mycobot_description/urdf/mech/mycobot_280_arm.urdf.xacro (robot description, xacro)
@@ -1,8 +1,9 @@
 <?xml version="1.0"?>
 <robot xmlns:xacro="http://www.ros.org/wiki/xacro">
-  <xacro:property name="joint_effort" value="56.0"/>
-  <xacro:property name="joint_velocity" value="2.792527"/>
-  <xacro:property name="joint_damping" value="0.0"/>
-  <xacro:property name="joint_friction" value="0.0"/>
+  <xacro:property name="joint_effort" value="56.0"/> <!-- This is the maximum force the joint can exert which is the maxmum torque the joint can apply-->
+  <xacro:property name="joint_velocity" value="2.792527"/> <!-- This is the maximum joint velocity in raians per second-->
+  <xacro:property name="joint_damping" value="0.0"/> <!-- Joint dampping coefficient -->
+  <xacro:property name="joint_friction" value="0.0"/> <!-- Joint friction coefficient-->
+  <!--here we got the masses for each links of our robotic arm  -->
   <xacro:property name="link1_mass" value="0.12"/>
   <xacro:property name="link2_mass" value="0.19"/>
@@ -11,5 +12,7 @@
   <xacro:property name="link5_mass" value="0.11"/>
   <xacro:property name="link6_mass" value="0.0739"/>
-  <xacro:property name="flange_mass" value="0.035"/>
+  <xacro:property name="flange_mass" value="0.035"/> <!-- This the last peiese the one that conected to the last link and this one is the one that conect the robotic arm with the gripper-->
+  <!-- A macro for the link_inertial and it's a plate for defining the inertial properties of links and we put it here in a macro so we don't repeat this block right here for every single link-->
+  <!-- The purpose of Shakro is to make sure that your URDF files stay nice and maintainable-->
   <xacro:macro name="link_inertial" params="mass ixx iyy izz">
     <inertial>
@@ -22,4 +25,5 @@
     </inertial>
   </xacro:macro>
+  <!-- This xacro macro handle the visual properties. Specifically how will each link appear in gazebo simulation.-->
   <xacro:macro name="material_visual" params="ref_link ambient diffuse specular">
     <gazebo reference="${ref_link}">
@@ -33,8 +37,10 @@
     </gazebo>
   </xacro:macro>
+  <!-- This xacro macro is the main robotic arm definition and this macros is called my_cobot_280_arm and it accepts these parameters the base_link, flange_link, prefix and origin -->
   <xacro:macro name="mycobot_280_arm" params="base_link flange_link prefix *origin">
-    <link name="${prefix}link1">
-      <xacro:link_inertial mass="${link1_mass}" ixx="0.000148" iyy="0.000148" izz="0.000096"/>
-      <visual>
+    <!-- So for each link form link1 through link6 plus the flang -->
+    <link name="${prefix}link1"> <!-- We define the link name -->
+      <xacro:link_inertial mass="${link1_mass}" ixx="0.000148" iyy="0.000148" izz="0.000096"/> <!-- The physical properties using link inertial macros-->
+      <visual> <!-- The visula properties and we tag the appropriate mesh file to define how this will actually look-->
         <geometry>
           <mesh filename="file://$(find mycobot_description)/meshes/mycobot_280/visual/link1.dae"/>
@@ -43,5 +49,5 @@
       </visual>
       <collision>
-        <geometry>
+        <geometry> <!-- And then simplify box geometry length,width and height for actual collision detection-->
           <box size="0.08 0.12 0.075"/>
         </geometry>
@@ -139,16 +145,17 @@
       </collision>
     </link>
-    <joint name="${prefix}${base_link}_to_${prefix}link1" type="fixed">
-      <parent link="${prefix}${base_link}"/>
-      <child link="${prefix}link1"/>
+    <!-- Now we get to the joints and joint conect all those link together-->
+    <joint name="${prefix}${base_link}_to_${prefix}link1" type="fixed"> <!-- This is the name of the joint and it tell us what this joint conect and the type of the joint is fixed because there's no motion in the base linke-->
+      <parent link="${prefix}${base_link}"/> <!-- Is the link that have the joint we want to conect it with other link-->
+      <child link="${prefix}link1"/> <!-- Is the link we want it to conect it with the link that have the joint -->
       <xacro:insert_block name="origin"/>
     </joint>
-    <joint name="${prefix}link1_to_${prefix}link2" type="revolute">
-      <axis xyz="0 0 1"/>
-      <limit effort="${joint_effort}" lower="-2.879793" upper="2.879793" velocity="${joint_velocity}"/>
+    <joint name="${prefix}link1_to_${prefix}link2" type="revolute"> <!-- But in this joint the type is revolute because it rotate so it's not fixed-->
+      <axis xyz="0 0 1"/> <!-- This define the axis of rotation the position of the rotation the joint will do in which axises and here mean we have rotation around the Z axis of the parent coordinate frame -->
+      <limit effort="${joint_effort}" lower="-2.879793" upper="2.879793" velocity="${joint_velocity}"/> <!-- This define the motion limits and this include the joint_effort which is the maximum torque the joint can apply. And we got the lower and upper which are the range of allowerd angles in radians and last we have the maximum angular velocity-->
       <parent link="${prefix}link1"/>
       <child link="${prefix}link2"/>
-      <origin xyz="0 0 0.13156" rpy="0 0 ${pi/2}"/>
-      <dynamics damping="${joint_damping}" friction="${joint_friction}"/>
+      <origin xyz="0 0 0.13156" rpy="0 0 ${pi/2}"/> <!-- This is the origin the position and orientation of the joint relative to the parent link-->
+      <dynamics damping="${joint_damping}" friction="${joint_friction}"/> <!-- Here we have damping and damping is the parameter measured in Newton meters per radian per second. And this determines how much the joint moving at a certain speed -->
     </joint>
     <joint name="${prefix}link2_to_${prefix}link3" type="revolute">
@@ -192,4 +199,5 @@
       <dynamics damping="${joint_damping}" friction="${joint_friction}"/>
     </joint>
+    <!-- Here we set the visual properties for each link and how it should look in Gazebo. 0.5 stand for color gray and 1 stand for color white.-->
     <xacro:material_visual ref_link="${prefix}link1" ambient="0.5 0.5 0.5 1" diffuse="0.5 0.5 0.5 1" specular="0.5 0.5 0.5 1"/>
     <xacro:material_visual ref_link="${prefix}link2" ambient="1 1 1 1" diffuse="1 1 1 1" specular="1 1 1 1"/>

File: mycobot_description/urdf/robots/mycobot_280.urdf.xacro (robot description, xacro)
@@ -1,14 +1,19 @@
 <?xml version="1.0"?>
 <robot xmlns:xacro="http://www.ros.org/wiki/xacro" name="mycobot_280">
+    <!-- This modular approach make it easier to swap our different bases or grippers or creaet multiple robot with different configurations or if we going to create a humanoid robot and we want to have a left arm and right arm
+    it's very modular and very flexible and allows us to do that-->
+    <!-- THIS FILES IS THE FILE THAT BRINGS ALL THOSE COMPONENETS TOGETHER. -->
     <xacro:arg name="robot_name" default="mycobot_280"/>
-    <xacro:arg name="add_world" default="true"/>
-    <xacro:arg name="base_link" default="base_link"/>
-    <xacro:arg name="base_type" default="g_shape"/>
-    <xacro:arg name="flange_link" default="link6_flange"/>
-    <xacro:arg name="gripper_type" default="adaptive_gripper"/>
-    <xacro:arg name="prefix" default=""/>
+    <xacro:arg name="add_world" default="true"/> <!-- This for adding a world link for our URDF-->
+    <xacro:arg name="base_link" default="base_link"/> <!-- The name of the base link of the robotic arm-->
+    <xacro:arg name="base_type" default="g_shape"/> <!-- The type of the base to use-->
+    <xacro:arg name="flange_link" default="link6_flange"/> <!-- The name of the endeffector the end link of the arm-->
+    <xacro:arg name="gripper_type" default="adaptive_gripper"/> <!-- This the name of the gripper we are using-->
+    <xacro:arg name="prefix" default=""/> <!-- This going to be blank but if you deal with dual arm robot link in humaind robot you can name it because we need one for the left arm and one for the right arm-->
     <xacro:arg name="use_camera" default="false"/>
     <xacro:arg name="use_gazebo" default="false"/>
-    <xacro:arg name="use_gripper" default="true"/>
+    <xacro:arg name="use_gripper" default="true"/> <!-- Here you can remove the gripper if you don't want to use it in the simulation-->
+    <!-- This say if the add_world parameter is true we need to create a world link to conect our robot to it. And that's like a vertual joint not like real physical joint.
+     it's just a vertual joint between the robot and the base link of the robotic arm. And it's connected at the origin of the world, The base link is conected to the origin of the world. -->
     <xacro:if value="$(arg add_world)">
       <link name="world"/>
@@ -19,4 +24,5 @@
       </joint>
     </xacro:if>
+    <!-- Here we handle the base the g_shape the gray platform to which we conect our robot to. We need to include it right here. But if you don't want this g_shape base so you will not need to include it. -->
     <xacro:property name="current_base" value="$(arg base_type)"/>
     <xacro:if value="${current_base == 'g_shape'}">
@@ -33,4 +39,5 @@
       <origin xyz="0 0 0" rpy="0 0 0"/>
     </xacro:mycobot_280_arm>
+    <!-- This is the gripper we added it here becaue we are using a gripper-->
     <xacro:if value="$(arg use_gripper)">
         <xacro:property name="current_gripper" value="$(arg gripper_type)"/>
@@ -44,13 +51,3 @@
         </xacro:if>
     </xacro:if>
-    <xacro:include filename="$(find mycobot_description)/urdf/control/gazebo_sim_ros2_control.urdf.xacro" />
-    <xacro:load_gazebo_sim_ros2_control_plugin
-      robot_name="$(arg robot_name)"
-      use_gazebo="$(arg use_gazebo)"/>
-    <xacro:include filename="$(find mycobot_description)/urdf/control/mycobot_280_ros2_control.urdf.xacro" />
-    <xacro:mycobot_ros2_control
-      prefix="$(arg prefix)"
-      flange_link="$(arg flange_link)"
-      use_gazebo="$(arg use_gazebo)"/>
-    <xacro:include filename="$(find mycobot_description)/urdf/sensors/intel_rgbd_cam_d435.urdf.xacro"/>
 </robot>
